File: files/KiCAD_files/JOLT_V1.kicad_pcb (KiCad board)
At the start: 2 copper layers, 71.8 x 48.5 mm, 73 parts, among them J1 Conn_01x04_Pin, J13 Conn_01x05_Pin, J2 Conn_01x10_Socket, J3 Conn_01x04_Pin, J4 XT60-M, J5 Conn_01x13_Socket, SW1 SW_Push, SW2 SW_SPDT, U1 STM32F405RGT6, U2 AMS1117-3.3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

Commit message: Add modified files
Other:
- board text added: "0"
- board text added: "1"
- board text added: "10"
- board text added: "11"
- board text added: "12"
- board text added: "13"
- board text added: "14"
- board text added: "15"
- board text added: "16"
- board text added: "17"
- board text added: "18"
- board text added: "19"
- board text added: "2"
- board text added: "20"
- board text added: "21"
- board text added: "22"
- board text added: "3"
- board text added: "4"
- board text added: "5"
- board text added: "6"
- board text added: "7"
- board text added: "8"
- board text added: "9"
- board text added: "Designed by Shaurya Tamang github.com/GoTouchGra55"
- board text added: "STRIDE v1.0"
